File: Hardware/USB-C PSU.kicad_sch (KiCad schematic)
At the start: 53 parts, among them J1 USB_C_Receptacle_USB2.0_16P, J2 VOUT, J3 TC2030, J4 VIN, SW1 SW_Reverse, SW2 Boot, SW3 Reset, U1 CH32X035G8U6, U4 LMR51610XDBVR, U5 TPD4S480RUKR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

Commit message: final tweaks before routing traces
Parts:
- added TP21: TestPoint, TestPoint:TestPoint_Pad_D1.0mm, symbol Connector:TestPoint
Connections:
- net +5V: now also TP21.1
Changed lines of the file:
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@@
 	(wire
 		(pts
+			(xy 259.08 63.5) (xy 267.97 63.5)
+		)
+		(stroke
+			(width 0)
+			(type default)
+		)
+	)
+	(wire
+		(pts
 			(xy 38.1 170.18) (xy 38.1 171.45)
 		)
@@
 	(label "C_D-"
 		(at 53.34 46.99 0)
-		(fields_autoplaced yes)
 		(effects
 			(font
@@
 	(label "BUCK_VIN"
 		(at 201.93 137.16 0)
-		(fields_autoplaced yes)
 		(effects
 			(font
@@
 	(label "C_D+"
 		(at 53.34 52.07 0)
-		(fields_autoplaced yes)
 		(effects
 			(font
@@
 	(label "C_CC2"
 		(at 53.34 40.64 0)
-		(fields_autoplaced yes)
 		(effects
 			(font
@@
 	(label "C_CC1"
 		(at 53.34 38.1 0)
-		(fields_autoplaced yes)
 		(effects
 			(font
@@
 	)
 	(symbol
+		(lib_id "Connector:TestPoint")
+		(at 267.97 63.5 270)
+		(unit 1)
+		(exclude_from_sim no)
+		(in_bom yes)
+		(on_board yes)
+		(dnp no)
+		(property "Reference" "TP21"
+			(at 272.796 63.5 90)
+			(effects
+				(font
+					(size 1.27 1.27)
+				)
+				(justify left)
+			)
+		)
+		(property "Value" "TestPoint"
+			(at 278.638 63.5 90)
+			(effects
+				(font
+					(size 1.27 1.27)
+				)
+				(justify left)
+				(hide yes)
+			)
+		)
+		(property "Footprint" "TestPoint:TestPoint_Pad_D1.0mm"
+			(at 267.97 68.58 0)
+			(effects
+				(font
+					(size 1.27 1.27)
+				)
+				(hide yes)
+			)
+		)
+		(property "Datasheet" "~"
+			(at 267.97 68.58 0)
+			(effects
+				(font
+					(size 1.27 1.27)
+				)
+				(hide yes)
+			)
+		)
+		(property "Description" "test point"
+			(at 267.97 63.5 0)
+			(effects
+				(font
+					(size 1.27 1.27)
+				)
+				(hide yes)
+			)
+		)
+		(property "LCSC" ""
+			(at 267.97 63.5 0)
+			(effects
+				(font
+					(size 1.27 1.27)
+				)
+				(hide yes)
+			)
+		)
+		(pin "1"
+		)
+		(instances
+			(project "USB-C PSU"
+				(path "/2795a064-4b14-4857-8c9a-fd2d32a5a222"
+					(reference "TP21")
+					(unit 1)
+				)
+			)
+		)
+	)
+	(symbol
 		(lib_id "power:GND")
 		(at 267.97 157.48 0)
@@
 					(unit 1)
 				)
+			)
+		)
+	)
+	(symbol
+		(lib_id "power:+5V")
+		(at 259.08 63.5 0)
+		(unit 1)
+		(exclude_from_sim no)
+		(in_bom yes)
+		(on_board yes)
+		(dnp no)
+		(fields_autoplaced yes)
+		(property "Reference" "#PWR0148"
+			(at 259.08 67.31 0)
+			(effects
+				(font
+					(size 1.27 1.27)
+				)
+				(hide yes)
+			)
+		)
+		(property "Value" "+5V"
+			(at 259.08 58.42 0)
+			(effects
+				(font
+					(size 1.27 1.27)
+				)
+			)
+		)
+		(property "Footprint" ""
+			(at 259.08 63.5 0)
+			(effects
+				(font
+					(size 1.27 1.27)
+				)
+				(hide yes)
+			)
+		)
+		(property "Datasheet" ""
+			(at 259.08 63.5 0)
+			(effects
+				(font
+					(size 1.27 1.27)
+				)
+				(hide yes)
+			)
+		)
+		(property "Description" "Power symbol creates a global label with name \"+5V\""
+			(at 259.08 63.5 0)
+			(effects
+				(font
+					(size 1.27 1.27)
+				)
+				(hide yes)
+			)
+		)
+		(pin "1"
+		)
+		(instances
+			(project "USB-C PSU"
+				(path "/2795a064-4b14-4857-8c9a-fd2d32a5a222"
+					(reference "#PWR0148")
+					(unit 1)
+				)

Commit message: oops, all vias
Parts:
- removed C12: 100n 100V, Capacitor_SMD:C_0402_1005Metric, symbol Device:C_Small
- C11: value 22u -> 22u 10V
- C13: value 4u7 100V -> 1u 100V; footprint Capacitor_SMD:C_0402_1005Metric -> Capacitor_SMD:C_0603_1608Metric
- J3: symbol Connector:Conn_ARM_SWD_TagConnect_TC2030-NL -> Connector_Generic:Conn_01x07; LCSC Part (none) -> C2881892
- TP14, TP15: now not fitted
- TP3, TP4: now not fitted; now left out of the parts list
Connections:
- net RX: now also J3.7 (Pin_7)
- net TX: now also J3.6 (Pin_6)
- no-connect marks 6 -> 5
Other:
- note added: "Should be 4.7uF, but only 0603 fits Should be fine^{tm}"
- moved on the sheet: C10, C11, D5, L2, R13, R14, U4

Commit message: design silkscreen markings + some polish
Parts:
- J3: LCSC Part C2881892 -> (none)
Changed lines of the file:
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@@
 			)
 		)
-		(property "LCSC Part" "C2881892"
+		(property "LCSC" ""
 			(at 224.79 31.75 0)
 			(effects

Commit message: final tweaks for v1.0
Parts:
- C11: LCSC Part (none) -> C86295
- J2: LCSC Part C431092 -> C431092
Changed lines of the file:
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@@
 			)
 		)
-		(property "LCSC Part" " C431092"
+		(property "LCSC Part" "C431092"
 			(at 137.16 101.6 0)
 			(effects
@@
 			)
 		)
+		(property "LCSC Part" ""
+			(at 85.09 90.17 0)
+			(effects
+				(font
+					(size 1.27 1.27)
+				)
+				(hide yes)
+			)
+		)
 		(pin "1"
 		)
@@
 			(at 271.78 146.05 0)
 			(effects
+				(font
+					(size 1.27 1.27)
+				)
+				(hide yes)
+			)
+		)
+		(property "LCSC Part" "C86295"
+			(at 271.78 146.05 0)
+			(effects
